Commit message: Refractored the URDF to take advantage of the similarity between fingers. Created a macro to reduce repeatable code

File: leap_description/assets/leap_hand/robot.urdf.xacro (robot description, xacro)
@@ -1,259 +1,5 @@
 <?xml version="1.0"?>
-<robot xmlns:xacro="http://www.ros.org/wiki/xacro" name="onshape">
-    <xacro:arg name="controllers_yaml" default=""/>
-    <ros2_control name="GazeboSimSystem" type="system">
-        <hardware>
-            <plugin>gz_ros2_control/GazeboSimSystem</plugin>
-        </hardware>
-        <joint name="0">
-            <command_interface name="position">
-                <param name="min">-3.14</param>
-                <param name="max">3.14</param>
-            </command_interface>
-            <state_interface name="position">
-                <param name="initial_value">0.0</param>
-            </state_interface>
-            <state_interface name="velocity"/>
-            <state_interface name="position"/>
-            <state_interface name="effort"/>
-        </joint>
-        <joint name="1">
-            <command_interface name="position">
-                <param name="min">-3.14</param>
-                <param name="max">3.14</param>
-            </command_interface>
-            <state_interface name="position">
-                <param name="initial_value">0.0</param>
-            </state_interface>
-            <state_interface name="velocity"/>
-            <state_interface name="position"/>
-            <state_interface name="effort"/>
-        </joint>
-        <joint name="2">
-            <command_interface name="position">
-                <param name="min">-3.14</param>
-                <param name="max">3.14</param>
-            </command_interface>
-            <state_interface name="position">
-                <param name="initial_value">0.0</param>
-            </state_interface>
-            <state_interface name="velocity"/>
-            <state_interface name="position"/>
-            <state_interface name="effort"/>
-        </joint>
-        <joint name="3">
-            <command_interface name="position">
-                <param name="min">-3.14</param>
-                <param name="max">3.14</param>
-            </command_interface>
-            <state_interface name="position">
-                <param name="initial_value">0.0</param>
-            </state_interface>
-            <state_interface name="velocity"/>
-            <state_interface name="position"/>
-            <state_interface name="effort"/>
-        </joint>
-        <joint name="4">
-            <command_interface name="position">
-                <param name="min">-3.14</param>
-                <param name="max">3.14</param>
-            </command_interface>
-            <state_interface name="position">
-                <param name="initial_value">0.0</param>
-            </state_interface>
-            <state_interface name="velocity"/>
-            <state_interface name="position"/>
-            <state_interface name="effort"/>
-        </joint>
-        <joint name="5">
-            <command_interface name="position">
-                <param name="min">-3.14</param>
-                <param name="max">3.14</param>
-            </command_interface>
-            <state_interface name="position">
-                <param name="initial_value">0.0</param>
-            </state_interface>
-            <state_interface name="velocity"/>
-            <state_interface name="position"/>
-            <state_interface name="effort"/>
-        </joint>
-        <joint name="6">
-            <command_interface name="position">
-                <param name="min">-3.14</param>
-                <param name="max">3.14</param>
-            </command_interface>
-            <state_interface name="position">
-                <param name="initial_value">0.0</param>
-            </state_interface>
-            <state_interface name="velocity"/>
-            <state_interface name="position"/>
-            <state_interface name="effort"/>
-        </joint>
-        <joint name="7">
-            <command_interface name="position">
-                <param name="min">-3.14</param>
-                <param name="max">3.14</param>
-            </command_interface>
-            <state_interface name="position">
-                <param name="initial_value">0.0</param>
-            </state_interface>
-            <state_interface name="velocity"/>
-            <state_interface name="position"/>
-            <state_interface name="effort"/>
-        </joint>
-        <joint name="8">
-            <command_interface name="position">
-                <param name="min">-3.14</param>
-                <param name="max">3.14</param>
-            </command_interface>
-            <state_interface name="position">
-                <param name="initial_value">0.0</param>
-            </state_interface>
-            <state_interface name="velocity"/>
-            <state_interface name="position"/>
-            <state_interface name="effort"/>
-        </joint>
-        <joint name="9">
-            <command_interface name="position">
-                <param name="min">-3.14</param>
-                <param name="max">3.14</param>
-            </command_interface>
-            <state_interface name="position">
-                <param name="initial_value">0.0</param>
-            </state_interface>
-            <state_interface name="velocity"/>
-            <state_interface name="position"/>
-            <state_interface name="effort"/>
-        </joint>
-        <joint name="10">
-            <command_interface name="position">
-                <param name="min">-3.14</param>
-                <param name="max">3.14</param>
-            </command_interface>
-            <state_interface name="position">
-                <param name="initial_value">0.0</param>
-            </state_interface>
-            <state_interface name="velocity"/>
-            <state_interface name="position"/>
-            <state_interface name="effort"/>
-        </joint>
-        <joint name="11">
-            <command_interface name="position">
-                <param name="min">-3.14</param>
-                <param name="max">3.14</param>
-            </command_interface>
-            <state_interface name="position">
-                <param name="initial_value">0.0</param>
-            </state_interface>
-            <state_interface name="velocity"/>
-            <state_interface name="position"/>
-            <state_interface name="effort"/>
-        </joint>
-        <joint name="12">
-            <command_interface name="position">
-                <param name="min">-3.14</param>
-                <param name="max">3.14</param>
-            </command_interface>
-            <state_interface name="position">
-                <param name="initial_value">0.0</param>
-            </state_interface>
-            <state_interface name="velocity"/>
-            <state_interface name="position"/>
-            <state_interface name="effort"/>
-        </joint>
-        <joint name="13">
-            <command_interface name="position">
-                <param name="min">-3.14</param>
-                <param name="max">3.14</param>
-            </command_interface>
-            <state_interface name="position">
-                <param name="initial_value">1.5707963267948958919</param>
-            </state_interface>
-            <state_interface name="velocity"/>
-            <state_interface name="position"/>
-            <state_interface name="effort"/>
-        </joint>
-        <joint name="14">
-            <command_interface name="position">
-                <param name="min">-3.14</param>
-                <param name="max">3.14</param>
-            </command_interface>
-            <state_interface name="position">
-                <param name="initial_value">0.0</param>
-            </state_interface>
-            <state_interface name="velocity"/>
-            <state_interface name="position"/>
-            <state_interface name="effort"/>
-        </joint>
-        <joint name="15">
-            <command_interface name="position">
-                <param name="min">-3.14</param>
-                <param name="max">3.14</param>
-            </command_interface>
-            <state_interface name="position">
-                <param name="initial_value">0.0</param>
-            </state_interface>
-            <state_interface name="velocity"/>
-            <state_interface name="position"/>
-            <state_interface name="effort"/>
-        </joint>
-    </ros2_control>
-    <gazebo>
-        <plugin filename="libgz_ros2_control-system.so" name="gz_ros2_control::GazeboSimROS2ControlPlugin">
-            <!-- <parameters>$(arg controllers_yaml)</parameters> -->
-            <parameters>/home/joel/distrobox/ros2-ubuntu/leap_ws/src/leap_control/leap_sim/config/leap_controller.yaml</parameters>
-        </plugin>
-    </gazebo>
-    <gazebo reference="palm_lower">
-        <selfCollide>true</selfCollide>
-    </gazebo>
-    <gazebo reference="mcp_joint">
-        <selfCollide>true</selfCollide>
-    </gazebo>
-    <gazebo reference="pip">
-        <selfCollide>true</selfCollide>
-    </gazebo>
-    <gazebo reference="dip">
-        <selfCollide>true</selfCollide>
-    </gazebo>
-    <gazebo reference="fingertip">
-        <selfCollide>true</selfCollide>
-    </gazebo>
-    <gazebo reference="mcp_joint_2">
-        <selfCollide>true</selfCollide>
-    </gazebo>
-    <gazebo reference="pip_2">
-        <selfCollide>true</selfCollide>
-    </gazebo>
-    <gazebo reference="dip_2">
-        <selfCollide>true</selfCollide>
-    </gazebo>
-    <gazebo reference="fingertip_2">
-        <selfCollide>true</selfCollide>
-    </gazebo>
-    <gazebo reference="mcp_joint_3">
-        <selfCollide>true</selfCollide>
-    </gazebo>
-    <gazebo reference="pip_3">
-        <selfCollide>true</selfCollide>
-    </gazebo>
-    <gazebo reference="dip_3">
-        <selfCollide>true</selfCollide>
-    </gazebo>
-    <gazebo reference="fingertip_3">
-        <selfCollide>true</selfCollide>
-    </gazebo>
-    <gazebo reference="thumb_pip">
-        <selfCollide>true</selfCollide>
-    </gazebo>
-    <gazebo reference="pip_4">
-        <selfCollide>true</selfCollide>
-    </gazebo>
-    <gazebo reference="thumb_dip">
-        <selfCollide>true</selfCollide>
-    </gazebo>
-    <gazebo reference="thumb_fingertip">
-        <selfCollide>true</selfCollide>
-    </gazebo>
+<robot xmlns:xacro="http://www.ros.org/wiki/xacro" name="leap">
+    <xacro:include filename="$(find leap_description)/assets/leap_hand/finger.xacro" />
     <link name="palm_lower">
         <visual>
@@ -261,9 +7,9 @@
                 rpy="0 -0 0" />
             <geometry>
-                <mesh filename="palm_lower.stl" />
+                <mesh filename="package://leap_description/assets/leap_hand/palm_lower.stl" />
             </geometry>
             <material name="palm_lower_material">
                 <color
-                    rgba="0.60392156862745094426 0.14901960784313725283 0.14901960784313725283 1.0" />
+                    rgba="1 1 1 1.0" />
             </material>
         </visual>
@@ -272,5 +18,5 @@
                 rpy="0 -0 0" />
             <geometry>
-                <mesh filename="palm_lower.stl" />
+                <mesh filename="package://leap_description/assets/leap_hand/palm_lower.stl" />
             </geometry>
         </collision>
@@ -282,49 +28,29 @@
         </inertial>
     </link>
-    <link name="mcp_joint">
-        <visual>
-            <origin xyz="0.0084069022611744960438 0.0077662438597169954416 0.014657354985032912051"
-                rpy="1.6375789613220999807e-15 -1.0210473302491019535e-30 1.7177968783327987474e-31" />
-            <geometry>
-                <mesh filename="mcp_joint.stl" />
-            </geometry>
-            <material name="mcp_joint_material">
-                <color
-                    rgba="0.86666666666666669627 0.86666666666666669627 0.050980392156862744391 1.0" />
-            </material>
-        </visual>
-        <collision>
-            <origin xyz="0.0084069022611744960438 0.0077662438597169954416 0.014657354985032912051"
-                rpy="1.6375789613220999807e-15 -1.0210473302491019535e-30 1.7177968783327987474e-31" />
-            <geometry>
-                <mesh filename="mcp_joint.stl" />
-            </geometry>
-        </collision>
-        <inertial>
-            <origin xyz="0 0 0" rpy="0 0 0" />
-            <mass value="0.044" />
-            <inertia ixx="0.000011499" ixy="0.000003049" ixz="0.000000121" iyy="0.000007796"
-                iyz="0.000000112" izz="0.000014759" />
-        </inertial>
-    </link>
-    <link name="pip">
+    <xacro:finger_template finger="index" root="palm_lower" x="-0.0070952496528625457958"
+        y="0.023057756134899472233" z="-0.01872240357846021927" />
+    <xacro:finger_template finger="middle" root="palm_lower" x="-0.0070952496528625457958"
+        y="-0.022392243865100525113" z="-0.01872240357846021927" />
+    <xacro:finger_template finger="ring" root="palm_lower" x="-0.0070952496528625457958"
+        y="-0.067842243865100515521" z="-0.01872240357846021927" />
+    <link name="thumb_semi_palm_1">
         <visual>
             <origin
-                xyz="0.0096433630922713280131 0.00029999999999998951117 0.00078403401041737645627"
+                xyz="-0.005356 0.0003 0.000784"
                 rpy="-1.570796326794896558 -1.570796326794896336 0" />
             <geometry>
-                <mesh filename="pip.stl" />
+                <mesh filename="package://leap_description/assets/leap_hand/proximal_phalanx_2.stl" />
             </geometry>
-            <material name="pip_material">
+            <material name="thumb_semi_palm_2_material">
                 <color
-                    rgba="0.74901960784313725839 0.74901960784313725839 0.74901960784313725839 1.0" />
+                    rgba="0 0 0 1.0" />
             </material>
         </visual>
         <collision>
             <origin
-                xyz="0.0096433630922713280131 0.00029999999999998951117 0.00078403401041737645627"
+                xyz="-0.005356 0.0003 0.000784"
                 rpy="-1.570796326794896558 -1.570796326794896336 0" />
             <geometry>
-                <mesh filename="pip.stl" />
+                <mesh filename="package://leap_description/assets/leap_hand/proximal_phalanx_2.stl" />
             </geometry>
         </collision>
@@ -336,423 +62,23 @@
         </inertial>
     </link>
-    <link name="dip">
-        <visual>
-            <origin xyz="0.021133352895225002849 -0.0084321191467048792201 0.0097850881620952408213"
-                rpy="-3.141592653589793116 4.5075111242164408299e-32 4.4395481053923607589e-32" />
-            <geometry>
-                <mesh filename="dip.stl" />
-            </geometry>
-            <material name="dip_material">
-                <color
-                    rgba="0.86666666666666669627 0.86666666666666669627 0.050980392156862744391 1.0" />
-            </material>
-        </visual>
-        <collision>
-            <origin xyz="0.021133352895225002849 -0.0084321191467048792201 0.0097850881620952408213"
-                rpy="-3.141592653589793116 4.5075111242164408299e-32 4.4395481053923607589e-32" />
-            <geometry>
-                <mesh filename="dip.stl" />
-            </geometry>
-        </collision>
-        <inertial>
-            <origin xyz="0 0 0" rpy="0 0 0" />
-            <mass value="0.037" />
-            <inertia ixx="0.000005542" ixy="-0.000000607" ixz="-0.000000017" iyy="0.000005727"
-                iyz="-0.000000023" izz="0.000006682" />
-        </inertial>
-    </link>
-    <link name="fingertip">
-        <visual>
-            <origin xyz="0.013286424108533503169 -0.0061142383865419869249 0.014499999999999497666"
-                rpy="3.141592653589793116 1.1993117970061734707e-33 4.4395481053923607589e-32" />
-            <geometry>
-                <mesh filename="fingertip.stl" />
-            </geometry>
-            <material name="fingertip_material">
-                <color
-                    rgba="0.86666666666666669627 0.86666666666666669627 0.050980392156862744391 1.0" />
-            </material>
-        </visual>
-        <collision>
-            <origin xyz="0.013286424108533503169 -0.0061142383865419869249 0.014499999999999497666"
-                rpy="3.141592653589793116 1.1993117970061734707e-33 4.4395481053923607589e-32" />
-            <geometry>
-                <mesh filename="fingertip.stl" />
-            </geometry>
-        </collision>
-        <inertial>
-            <origin xyz="0 0 0" rpy="0 0 0" />
-            <mass value="0.016" />
-            <inertia ixx="0.000003368" ixy="0.000000115" ixz="0" iyy="0.000001556" iyz="0"
-                izz="0.000002863" />
-        </inertial>
-    </link>
-    <joint name="0" type="revolute">
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