Commit message: Refractored the URDF to take advantage of the similarity between fingers. Created a macro to reduce repeatable code

File: leap_description/assets/leap_hand/robot_gz.urdf.xacro (robot description, xacro)
@@ -1,4 +1,259 @@
 <?xml version="1.0"?>
-<robot xmlns:xacro="http://www.ros.org/wiki/xacro" name="leap">
+<robot xmlns:xacro="http://www.ros.org/wiki/xacro" name="onshape">
+    <xacro:arg name="controllers_yaml" default=""/>
+    <ros2_control name="GazeboSimSystem" type="system">
+        <hardware>
+            <plugin>gz_ros2_control/GazeboSimSystem</plugin>
+        </hardware>
+        <joint name="0">
+            <command_interface name="position">
+                <param name="min">-3.14</param>
+                <param name="max">3.14</param>
+            </command_interface>
+            <state_interface name="position">
+                <param name="initial_value">0.0</param>
+            </state_interface>
+            <state_interface name="velocity"/>
+            <state_interface name="position"/>
+            <state_interface name="effort"/>
+        </joint>
+        <joint name="1">
+            <command_interface name="position">
+                <param name="min">-3.14</param>
+                <param name="max">3.14</param>
+            </command_interface>
+            <state_interface name="position">
+                <param name="initial_value">0.0</param>
+            </state_interface>
+            <state_interface name="velocity"/>
+            <state_interface name="position"/>
+            <state_interface name="effort"/>
+        </joint>
+        <joint name="2">
+            <command_interface name="position">
+                <param name="min">-3.14</param>
+                <param name="max">3.14</param>
+            </command_interface>
+            <state_interface name="position">
+                <param name="initial_value">0.0</param>
+            </state_interface>
+            <state_interface name="velocity"/>
+            <state_interface name="position"/>
+            <state_interface name="effort"/>
+        </joint>
+        <joint name="3">
+            <command_interface name="position">
+                <param name="min">-3.14</param>
+                <param name="max">3.14</param>
+            </command_interface>
+            <state_interface name="position">
+                <param name="initial_value">0.0</param>
+            </state_interface>
+            <state_interface name="velocity"/>
+            <state_interface name="position"/>
+            <state_interface name="effort"/>
+        </joint>
+        <joint name="4">
+            <command_interface name="position">
+                <param name="min">-3.14</param>
+                <param name="max">3.14</param>
+            </command_interface>
+            <state_interface name="position">
+                <param name="initial_value">0.0</param>
+            </state_interface>
+            <state_interface name="velocity"/>
+            <state_interface name="position"/>
+            <state_interface name="effort"/>
+        </joint>
+        <joint name="5">
+            <command_interface name="position">
+                <param name="min">-3.14</param>
+                <param name="max">3.14</param>
+            </command_interface>
+            <state_interface name="position">
+                <param name="initial_value">0.0</param>
+            </state_interface>
+            <state_interface name="velocity"/>
+            <state_interface name="position"/>
+            <state_interface name="effort"/>
+        </joint>
+        <joint name="6">
+            <command_interface name="position">
+                <param name="min">-3.14</param>
+                <param name="max">3.14</param>
+            </command_interface>
+            <state_interface name="position">
+                <param name="initial_value">0.0</param>
+            </state_interface>
+            <state_interface name="velocity"/>
+            <state_interface name="position"/>
+            <state_interface name="effort"/>
+        </joint>
+        <joint name="7">
+            <command_interface name="position">
+                <param name="min">-3.14</param>
+                <param name="max">3.14</param>
+            </command_interface>
+            <state_interface name="position">
+                <param name="initial_value">0.0</param>
+            </state_interface>
+            <state_interface name="velocity"/>
+            <state_interface name="position"/>
+            <state_interface name="effort"/>
+        </joint>
+        <joint name="8">
+            <command_interface name="position">
+                <param name="min">-3.14</param>
+                <param name="max">3.14</param>
+            </command_interface>
+            <state_interface name="position">
+                <param name="initial_value">0.0</param>
+            </state_interface>
+            <state_interface name="velocity"/>
+            <state_interface name="position"/>
+            <state_interface name="effort"/>
+        </joint>
+        <joint name="9">
+            <command_interface name="position">
+                <param name="min">-3.14</param>
+                <param name="max">3.14</param>
+            </command_interface>
+            <state_interface name="position">
+                <param name="initial_value">0.0</param>
+            </state_interface>
+            <state_interface name="velocity"/>
+            <state_interface name="position"/>
+            <state_interface name="effort"/>
+        </joint>
+        <joint name="10">
+            <command_interface name="position">
+                <param name="min">-3.14</param>
+                <param name="max">3.14</param>
+            </command_interface>
+            <state_interface name="position">
+                <param name="initial_value">0.0</param>
+            </state_interface>
+            <state_interface name="velocity"/>
+            <state_interface name="position"/>
+            <state_interface name="effort"/>
+        </joint>
+        <joint name="11">
+            <command_interface name="position">
+                <param name="min">-3.14</param>
+                <param name="max">3.14</param>
+            </command_interface>
+            <state_interface name="position">
+                <param name="initial_value">0.0</param>
+            </state_interface>
+            <state_interface name="velocity"/>
+            <state_interface name="position"/>
+            <state_interface name="effort"/>
+        </joint>
+        <joint name="12">
+            <command_interface name="position">
+                <param name="min">-3.14</param>
+                <param name="max">3.14</param>
+            </command_interface>
+            <state_interface name="position">
+                <param name="initial_value">0.0</param>
+            </state_interface>
+            <state_interface name="velocity"/>
+            <state_interface name="position"/>
+            <state_interface name="effort"/>
+        </joint>
+        <joint name="13">
+            <command_interface name="position">
+                <param name="min">-3.14</param>
+                <param name="max">3.14</param>
+            </command_interface>
+            <state_interface name="position">
+                <param name="initial_value">1.5707963267948958919</param>
+            </state_interface>
+            <state_interface name="velocity"/>
+            <state_interface name="position"/>
+            <state_interface name="effort"/>
+        </joint>
+        <joint name="14">
+            <command_interface name="position">
+                <param name="min">-3.14</param>
+                <param name="max">3.14</param>
+            </command_interface>
+            <state_interface name="position">
+                <param name="initial_value">0.0</param>
+            </state_interface>
+            <state_interface name="velocity"/>
+            <state_interface name="position"/>
+            <state_interface name="effort"/>
+        </joint>
+        <joint name="15">
+            <command_interface name="position">
+                <param name="min">-3.14</param>
+                <param name="max">3.14</param>
+            </command_interface>
+            <state_interface name="position">
+                <param name="initial_value">0.0</param>
+            </state_interface>
+            <state_interface name="velocity"/>
+            <state_interface name="position"/>
+            <state_interface name="effort"/>
+        </joint>
+    </ros2_control>
+    <gazebo>
+        <plugin filename="libgz_ros2_control-system.so" name="gz_ros2_control::GazeboSimROS2ControlPlugin">
+            <!-- <parameters>$(arg controllers_yaml)</parameters> -->
+            <parameters>/home/joel/distrobox/ros2-ubuntu/leap_ws/src/leap_control/leap_sim/config/leap_controller.yaml</parameters>
+        </plugin>
+    </gazebo>
+    <gazebo reference="palm_lower">
+        <selfCollide>true</selfCollide>
+    </gazebo>
+    <gazebo reference="mcp_joint">
+        <selfCollide>true</selfCollide>
+    </gazebo>
+    <gazebo reference="pip">
+        <selfCollide>true</selfCollide>
+    </gazebo>
+    <gazebo reference="dip">
+        <selfCollide>true</selfCollide>
+    </gazebo>
+    <gazebo reference="fingertip">
+        <selfCollide>true</selfCollide>
+    </gazebo>
+    <gazebo reference="mcp_joint_2">
+        <selfCollide>true</selfCollide>
+    </gazebo>
+    <gazebo reference="pip_2">
+        <selfCollide>true</selfCollide>
+    </gazebo>
+    <gazebo reference="dip_2">
+        <selfCollide>true</selfCollide>
+    </gazebo>
+    <gazebo reference="fingertip_2">
+        <selfCollide>true</selfCollide>
+    </gazebo>
+    <gazebo reference="mcp_joint_3">
+        <selfCollide>true</selfCollide>
+    </gazebo>
+    <gazebo reference="pip_3">
+        <selfCollide>true</selfCollide>
+    </gazebo>
+    <gazebo reference="dip_3">
+        <selfCollide>true</selfCollide>
+    </gazebo>
+    <gazebo reference="fingertip_3">
+        <selfCollide>true</selfCollide>
+    </gazebo>
+    <gazebo reference="thumb_pip">
+        <selfCollide>true</selfCollide>
+    </gazebo>
+    <gazebo reference="pip_4">
+        <selfCollide>true</selfCollide>
+    </gazebo>
+    <gazebo reference="thumb_dip">
+        <selfCollide>true</selfCollide>
+    </gazebo>
+    <gazebo reference="thumb_fingertip">
+        <selfCollide>true</selfCollide>
+    </gazebo>
     <link name="palm_lower">
         <visual>
@@ -6,9 +261,9 @@
                 rpy="0 -0 0" />
             <geometry>
-                <mesh filename="package://leap_description/assets/leap_hand/palm_lower.stl" />
+                <mesh filename="palm_lower.stl" />
             </geometry>
             <material name="palm_lower_material">
                 <color
-                    rgba="1 1 1 1.0" />
+                    rgba="0.60392156862745094426 0.14901960784313725283 0.14901960784313725283 1.0" />
             </material>
         </visual>
@@ -17,5 +272,5 @@
                 rpy="0 -0 0" />
             <geometry>
-                <mesh filename="package://leap_description/assets/leap_hand/palm_lower.stl" />
+                <mesh filename="palm_lower.stl" />
             </geometry>
         </collision>
@@ -27,14 +282,14 @@
         </inertial>
     </link>
-    <link name="index_proximal_phalanx_1">
+    <link name="mcp_joint">
         <visual>
             <origin xyz="0.0084069022611744960438 0.0077662438597169954416 0.014657354985032912051"
                 rpy="1.6375789613220999807e-15 -1.0210473302491019535e-30 1.7177968783327987474e-31" />
             <geometry>
-                <mesh filename="package://leap_description/assets/leap_hand/mcp_joint.stl" />
+                <mesh filename="mcp_joint.stl" />
             </geometry>
             <material name="mcp_joint_material">
                 <color
-                    rgba="0 0 0 1.0" />
+                    rgba="0.86666666666666669627 0.86666666666666669627 0.050980392156862744391 1.0" />
             </material>
         </visual>
@@ -43,5 +298,5 @@
                 rpy="1.6375789613220999807e-15 -1.0210473302491019535e-30 1.7177968783327987474e-31" />
             <geometry>
-                <mesh filename="package://leap_description/assets/leap_hand/mcp_joint.stl" />
+                <mesh filename="mcp_joint.stl" />
             </geometry>
         </collision>
@@ -53,5 +308,5 @@
         </inertial>
     </link>
-    <link name="index_proximal_phalanx_2">
+    <link name="pip">
         <visual>
             <origin
@@ -59,9 +314,9 @@
                 rpy="-1.570796326794896558 -1.570796326794896336 0" />
             <geometry>
-                <mesh filename="package://leap_description/assets/leap_hand/pip.stl" />
+                <mesh filename="pip.stl" />
             </geometry>
             <material name="pip_material">
                 <color
-                    rgba="0 0 0 1.0" />
+                    rgba="0.74901960784313725839 0.74901960784313725839 0.74901960784313725839 1.0" />
             </material>
         </visual>
@@ -71,5 +326,5 @@
                 rpy="-1.570796326794896558 -1.570796326794896336 0" />
             <geometry>
-                <mesh filename="package://leap_description/assets/leap_hand/pip.stl" />
+                <mesh filename="pip.stl" />
             </geometry>
         </collision>
@@ -81,14 +336,14 @@
         </inertial>
     </link>
-    <link name="index_middle_phalanx">
+    <link name="dip">
         <visual>
             <origin xyz="0.021133352895225002849 -0.0084321191467048792201 0.0097850881620952408213"
                 rpy="-3.141592653589793116 4.5075111242164408299e-32 4.4395481053923607589e-32" />
             <geometry>
-                <mesh filename="package://leap_description/assets/leap_hand/dip.stl" />
+                <mesh filename="dip.stl" />
             </geometry>
             <material name="dip_material">
                 <color
-                    rgba="0 0 0 1.0" />
+                    rgba="0.86666666666666669627 0.86666666666666669627 0.050980392156862744391 1.0" />
             </material>
         </visual>
@@ -97,5 +352,5 @@
                 rpy="-3.141592653589793116 4.5075111242164408299e-32 4.4395481053923607589e-32" />
             <geometry>
-                <mesh filename="package://leap_description/assets/leap_hand/dip.stl" />
+                <mesh filename="dip.stl" />
             </geometry>
         </collision>
@@ -107,14 +362,14 @@
         </inertial>
     </link>
-    <link name="index_distal_phalanx">
+    <link name="fingertip">
         <visual>
             <origin xyz="0.013286424108533503169 -0.0061142383865419869249 0.014499999999999497666"
                 rpy="3.141592653589793116 1.1993117970061734707e-33 4.4395481053923607589e-32" />
             <geometry>
-                <mesh filename="package://leap_description/assets/leap_hand/fingertip.stl" />
+                <mesh filename="fingertip.stl" />
             </geometry>
             <material name="fingertip_material">
                 <color
-                    rgba="1 1 1 1.0" />
+                    rgba="0.86666666666666669627 0.86666666666666669627 0.050980392156862744391 1.0" />
             </material>
         </visual>
@@ -123,5 +378,5 @@
                 rpy="3.141592653589793116 1.1993117970061734707e-33 4.4395481053923607589e-32" />
             <geometry>
-                <mesh filename="package://leap_description/assets/leap_hand/fingertip.stl" />
+                <mesh filename="fingertip.stl" />
             </geometry>
         </collision>
@@ -133,46 +388,46 @@
         </inertial>
     </link>
-    <joint name="index_pip_flex_joint" type="revolute">
+    <joint name="0" type="revolute">
         <origin xyz="-0.0070952496528625457958 0.023057756134899472233 -0.01872240357846021927"
             rpy="1.5707963267948950037 1.5707963267948945596 0" />
         <parent link="palm_lower" />
-        <child link="index_proximal_phalanx_1" />
+        <child link="mcp_joint" />
         <axis xyz="0 0 -1" />
         <limit effort="0.95" velocity="8.48" lower="-0.314" upper="2.23" />
         <joint_properties friction="0.0" />
     </joint>
-    <joint name="index_pip_abb_joint" type="revolute">
+    <joint name="1" type="revolute">
         <origin xyz="-0.012200000000000007713 0.038099999999999994982 0.014500000000000000736"
             rpy="-1.570796326794896558 -1.0065212660796336576e-15 1.5707963267948943376" />
-        <parent link="index_proximal_phalanx_1" />
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