Commit message: Started adapting the gazebo driver for moveit planning

File: leap_description/assets/leap_hand/robot_gz.urdf.xacro (robot description, xacro)
@@ -1,4 +1,4 @@
 <?xml version="1.0"?>
-<robot xmlns:xacro="http://www.ros.org/wiki/xacro" name="onshape">
+<robot xmlns:xacro="http://www.ros.org/wiki/xacro" name="leap">
     <xacro:arg name="controllers_yaml" default=""/>
     <ros2_control name="GazeboSimSystem" type="system">
@@ -6,161 +6,161 @@
             <plugin>gz_ros2_control/GazeboSimSystem</plugin>
         </hardware>
-        <joint name="0">
-            <command_interface name="position">
-                <param name="min">-3.14</param>
-                <param name="max">3.14</param>
-            </command_interface>
-            <state_interface name="position">
-                <param name="initial_value">0.0</param>
-            </state_interface>
-            <state_interface name="velocity"/>
-            <state_interface name="position"/>
-            <state_interface name="effort"/>
-        </joint>
-        <joint name="1">
-            <command_interface name="position">
-                <param name="min">-3.14</param>
-                <param name="max">3.14</param>
-            </command_interface>
-            <state_interface name="position">
-                <param name="initial_value">0.0</param>
-            </state_interface>
-            <state_interface name="velocity"/>
-            <state_interface name="position"/>
-            <state_interface name="effort"/>
-        </joint>
-        <joint name="2">
-            <command_interface name="position">
-                <param name="min">-3.14</param>
-                <param name="max">3.14</param>
-            </command_interface>
-            <state_interface name="position">
-                <param name="initial_value">0.0</param>
-            </state_interface>
-            <state_interface name="velocity"/>
-            <state_interface name="position"/>
-            <state_interface name="effort"/>
-        </joint>
-        <joint name="3">
-            <command_interface name="position">
-                <param name="min">-3.14</param>
-                <param name="max">3.14</param>
-            </command_interface>
-            <state_interface name="position">
-                <param name="initial_value">0.0</param>
-            </state_interface>
-            <state_interface name="velocity"/>
-            <state_interface name="position"/>
-            <state_interface name="effort"/>
-        </joint>
-        <joint name="4">
-            <command_interface name="position">
-                <param name="min">-3.14</param>
-                <param name="max">3.14</param>
-            </command_interface>
-            <state_interface name="position">
-                <param name="initial_value">0.0</param>
-            </state_interface>
-            <state_interface name="velocity"/>
-            <state_interface name="position"/>
-            <state_interface name="effort"/>
-        </joint>
-        <joint name="5">
-            <command_interface name="position">
-                <param name="min">-3.14</param>
-                <param name="max">3.14</param>
-            </command_interface>
-            <state_interface name="position">
-                <param name="initial_value">0.0</param>
-            </state_interface>
-            <state_interface name="velocity"/>
-            <state_interface name="position"/>
-            <state_interface name="effort"/>
-        </joint>
-        <joint name="6">
-            <command_interface name="position">
-                <param name="min">-3.14</param>
-                <param name="max">3.14</param>
-            </command_interface>
-            <state_interface name="position">
-                <param name="initial_value">0.0</param>
-            </state_interface>
-            <state_interface name="velocity"/>
-            <state_interface name="position"/>
-            <state_interface name="effort"/>
-        </joint>
-        <joint name="7">
-            <command_interface name="position">
-                <param name="min">-3.14</param>
-                <param name="max">3.14</param>
-            </command_interface>
-            <state_interface name="position">
-                <param name="initial_value">0.0</param>
-            </state_interface>
-            <state_interface name="velocity"/>
-            <state_interface name="position"/>
-            <state_interface name="effort"/>
-        </joint>
-        <joint name="8">
-            <command_interface name="position">
-                <param name="min">-3.14</param>
-                <param name="max">3.14</param>
-            </command_interface>
-            <state_interface name="position">
-                <param name="initial_value">0.0</param>
-            </state_interface>
-            <state_interface name="velocity"/>
-            <state_interface name="position"/>
-            <state_interface name="effort"/>
-        </joint>
-        <joint name="9">
-            <command_interface name="position">
-                <param name="min">-3.14</param>
-                <param name="max">3.14</param>
-            </command_interface>
-            <state_interface name="position">
-                <param name="initial_value">0.0</param>
-            </state_interface>
-            <state_interface name="velocity"/>
-            <state_interface name="position"/>
-            <state_interface name="effort"/>
-        </joint>
-        <joint name="10">
-            <command_interface name="position">
-                <param name="min">-3.14</param>
-                <param name="max">3.14</param>
-            </command_interface>
-            <state_interface name="position">
-                <param name="initial_value">0.0</param>
-            </state_interface>
-            <state_interface name="velocity"/>
-            <state_interface name="position"/>
-            <state_interface name="effort"/>
-        </joint>
-        <joint name="11">
-            <command_interface name="position">
-                <param name="min">-3.14</param>
-                <param name="max">3.14</param>
-            </command_interface>
-            <state_interface name="position">
-                <param name="initial_value">0.0</param>
-            </state_interface>
-            <state_interface name="velocity"/>
-            <state_interface name="position"/>
-            <state_interface name="effort"/>
-        </joint>
-        <joint name="12">
-            <command_interface name="position">
-                <param name="min">-3.14</param>
-                <param name="max">3.14</param>
-            </command_interface>
-            <state_interface name="position">
-                <param name="initial_value">0.0</param>
-            </state_interface>
-            <state_interface name="velocity"/>
-            <state_interface name="position"/>
-            <state_interface name="effort"/>
-        </joint>
-        <joint name="13">
+        <joint name="index_pip_flex_joint">
+            <command_interface name="position">
+                <param name="min">-3.14</param>
+                <param name="max">3.14</param>
+            </command_interface>
+            <state_interface name="position">
+                <param name="initial_value">0.0</param>
+            </state_interface>
+            <state_interface name="velocity"/>
+            <state_interface name="position"/>
+            <state_interface name="effort"/>
+        </joint>
+        <joint name="index_pip_abb_joint">
+            <command_interface name="position">
+                <param name="min">-3.14</param>
+                <param name="max">3.14</param>
+            </command_interface>
+            <state_interface name="position">
+                <param name="initial_value">0.0</param>
+            </state_interface>
+            <state_interface name="velocity"/>
+            <state_interface name="position"/>
+            <state_interface name="effort"/>
+        </joint>
+        <joint name="index_mcp_joint">
+            <command_interface name="position">
+                <param name="min">-3.14</param>
+                <param name="max">3.14</param>
+            </command_interface>
+            <state_interface name="position">
+                <param name="initial_value">0.0</param>
+            </state_interface>
+            <state_interface name="velocity"/>
+            <state_interface name="position"/>
+            <state_interface name="effort"/>
+        </joint>
+        <joint name="index_dip_joint">
+            <command_interface name="position">
+                <param name="min">-3.14</param>
+                <param name="max">3.14</param>
+            </command_interface>
+            <state_interface name="position">
+                <param name="initial_value">0.0</param>
+            </state_interface>
+            <state_interface name="velocity"/>
+            <state_interface name="position"/>
+            <state_interface name="effort"/>
+        </joint>
+        <joint name="middle_pip_flex_joint">
+            <command_interface name="position">
+                <param name="min">-3.14</param>
+                <param name="max">3.14</param>
+            </command_interface>
+            <state_interface name="position">
+                <param name="initial_value">0.0</param>
+            </state_interface>
+            <state_interface name="velocity"/>
+            <state_interface name="position"/>
+            <state_interface name="effort"/>
+        </joint>
+        <joint name="middle_pip_abb_joint">
+            <command_interface name="position">
+                <param name="min">-3.14</param>
+                <param name="max">3.14</param>
+            </command_interface>
+            <state_interface name="position">
+                <param name="initial_value">0.0</param>
+            </state_interface>
+            <state_interface name="velocity"/>
+            <state_interface name="position"/>
+            <state_interface name="effort"/>
+        </joint>
+        <joint name="middle_mcp_joint">
+            <command_interface name="position">
+                <param name="min">-3.14</param>
+                <param name="max">3.14</param>
+            </command_interface>
+            <state_interface name="position">
+                <param name="initial_value">0.0</param>
+            </state_interface>
+            <state_interface name="velocity"/>
+            <state_interface name="position"/>
+            <state_interface name="effort"/>
+        </joint>
+        <joint name="middle_dip_joint">
+            <command_interface name="position">
+                <param name="min">-3.14</param>
+                <param name="max">3.14</param>
+            </command_interface>
+            <state_interface name="position">
+                <param name="initial_value">0.0</param>
+            </state_interface>
+            <state_interface name="velocity"/>
+            <state_interface name="position"/>
+            <state_interface name="effort"/>
+        </joint>
+        <joint name="ring_pip_flex_joint">
+            <command_interface name="position">
+                <param name="min">-3.14</param>
+                <param name="max">3.14</param>
+            </command_interface>
+            <state_interface name="position">
+                <param name="initial_value">0.0</param>
+            </state_interface>
+            <state_interface name="velocity"/>
+            <state_interface name="position"/>
+            <state_interface name="effort"/>
+        </joint>
+        <joint name="ring_pip_abb_joint">
+            <command_interface name="position">
+                <param name="min">-3.14</param>
+                <param name="max">3.14</param>
+            </command_interface>
+            <state_interface name="position">
+                <param name="initial_value">0.0</param>
+            </state_interface>
+            <state_interface name="velocity"/>
+            <state_interface name="position"/>
+            <state_interface name="effort"/>
+        </joint>
+        <joint name="ring_mcp_joint">
+            <command_interface name="position">
+                <param name="min">-3.14</param>
+                <param name="max">3.14</param>
+            </command_interface>
+            <state_interface name="position">
+                <param name="initial_value">0.0</param>
+            </state_interface>
+            <state_interface name="velocity"/>
+            <state_interface name="position"/>
+            <state_interface name="effort"/>
+        </joint>
+        <joint name="ring_dip_joint">
+            <command_interface name="position">
+                <param name="min">-3.14</param>
+                <param name="max">3.14</param>
+            </command_interface>
+            <state_interface name="position">
+                <param name="initial_value">0.0</param>
+            </state_interface>
+            <state_interface name="velocity"/>
+            <state_interface name="position"/>
+            <state_interface name="effort"/>
+        </joint>
+        <joint name="thumb_cmc_abb_joint">
+            <command_interface name="position">
+                <param name="min">-3.14</param>
+                <param name="max">3.14</param>
+            </command_interface>
+            <state_interface name="position">
+                <param name="initial_value">0.0</param>
+            </state_interface>
+            <state_interface name="velocity"/>
+            <state_interface name="position"/>
+            <state_interface name="effort"/>
+        </joint>
+        <joint name="thumb_cmc_flex_joint">
             <command_interface name="position">
                 <param name="min">-3.14</param>
@@ -174,17 +174,17 @@
             <state_interface name="effort"/>
         </joint>
-        <joint name="14">
-            <command_interface name="position">
-                <param name="min">-3.14</param>
-                <param name="max">3.14</param>
-            </command_interface>
-            <state_interface name="position">
-                <param name="initial_value">0.0</param>
-            </state_interface>
-            <state_interface name="velocity"/>
-            <state_interface name="position"/>
-            <state_interface name="effort"/>
-        </joint>
-        <joint name="15">
+        <joint name="thumb_mcp_joint">
+            <command_interface name="position">
+                <param name="min">-3.14</param>
+                <param name="max">3.14</param>
+            </command_interface>
+            <state_interface name="position">
+                <param name="initial_value">0.0</param>
+            </state_interface>
+            <state_interface name="velocity"/>
+            <state_interface name="position"/>
+            <state_interface name="effort"/>
+        </joint>
+        <joint name="thumb_ip_joint">
             <command_interface name="position">
                 <param name="min">-3.14</param>
@@ -205,55 +205,5 @@
         </plugin>
     </gazebo>
-    <gazebo reference="palm_lower">
-        <selfCollide>true</selfCollide>
-    </gazebo>
-    <gazebo reference="mcp_joint">
-        <selfCollide>true</selfCollide>
-    </gazebo>
-    <gazebo reference="pip">
-        <selfCollide>true</selfCollide>
-    </gazebo>
-    <gazebo reference="dip">
-        <selfCollide>true</selfCollide>
-    </gazebo>
-    <gazebo reference="fingertip">
-        <selfCollide>true</selfCollide>
-    </gazebo>
-    <gazebo reference="mcp_joint_2">
-        <selfCollide>true</selfCollide>
-    </gazebo>
-    <gazebo reference="pip_2">
-        <selfCollide>true</selfCollide>
-    </gazebo>
-    <gazebo reference="dip_2">
-        <selfCollide>true</selfCollide>
-    </gazebo>
-    <gazebo reference="fingertip_2">
-        <selfCollide>true</selfCollide>
-    </gazebo>
-    <gazebo reference="mcp_joint_3">
-        <selfCollide>true</selfCollide>
-    </gazebo>
-    <gazebo reference="pip_3">
-        <selfCollide>true</selfCollide>
-    </gazebo>
-    <gazebo reference="dip_3">
-        <selfCollide>true</selfCollide>
-    </gazebo>
-    <gazebo reference="fingertip_3">
-        <selfCollide>true</selfCollide>
-    </gazebo>
-    <gazebo reference="thumb_pip">
-        <selfCollide>true</selfCollide>
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
File: leap_moveit/config/leap.urdf.xacro (robot description, xacro)
@@ -7,3 +7,9 @@
     <xacro:include filename="leap.ros2_control.xacro" />
     <xacro:leap_ros2_control name="FakeSystem" initial_positions_file="$(arg initial_positions_file)"/>
+    <gazebo>
+        <plugin filename="libgz_ros2_control-system.so" name="gz_ros2_control::GazeboSimROS2ControlPlugin">
+            <!-- <parameters>$(arg controllers_yaml)</parameters> -->
+            <parameters>/home/joel/distrobox/ros2-ubuntu/leap_ws/src/leap_control/leap_sim/config/leap_controller.yaml</parameters>
+        </plugin>
+    </gazebo>
 </robot>
