Commit message: Configured Moveit planning

File: leap_description/assets/leap_hand/finger.xacro (robot description, xacro)
@@ -120,5 +120,5 @@
             <child link="${finger}_proximal_phalanx_1" />
             <axis xyz="0 0 -1" />
-            <limit effort="0.95" velocity="8.48" lower="-0.314" upper="2.23" />
+            <limit effort="0.95" velocity="8.48" acceleration="20.0" lower="-0.314" upper="2.23" />
             <joint_properties friction="0.0" />
         </joint>
@@ -129,5 +129,5 @@
             <child link="${finger}_proximal_phalanx_2" />
             <axis xyz="0 0 -1" />
-            <limit effort="0.95" velocity="8.48" lower="-1.047" upper="1.047" />
+            <limit effort="0.95" velocity="8.48" acceleration="20.0" lower="-1.047" upper="1.047" />
             <joint_properties friction="0.0" />
         </joint>
@@ -138,5 +138,5 @@
             <child link="${finger}_middle_phalanx" />
             <axis xyz="0 0 -1" />
-            <limit effort="0.95" velocity="8.48" lower="-0.506" upper="1.885" />
+            <limit effort="0.95" velocity="8.48" acceleration="20.0" lower="-0.506" upper="1.885" />
             <joint_properties friction="0.0" />
         </joint>
@@ -148,5 +148,5 @@
             <child link="${finger}_distal_phalanx" />
             <axis xyz="0 0 -1" />
-            <limit effort="0.95" velocity="8.48" lower="-0.366" upper="2.042" />
+            <limit effort="0.95" velocity="8.48" acceleration="20.0" lower="-0.366" upper="2.042" />
             <joint_properties friction="0.0" />
         </joint>

File: leap_description/assets/leap_hand/robot.urdf.xacro (robot description, xacro)
@@ -151,5 +151,5 @@
         <child link="thumb_semi_palm_1" />
         <axis xyz="0 0 -1" />
-        <limit effort="0.95" velocity="8.48" lower="-0.349" upper="2.094" />
+        <limit effort="0.95" velocity="8.48" acceleration="20.0" lower="-0.349" upper="2.094" />
         <joint_properties friction="0.0" />
     </joint>
@@ -160,5 +160,5 @@
         <child link="thumb_semi_palm_2" />
         <axis xyz="0 0 -1" />
-        <limit effort="0.95" velocity="8.48" lower="-2.47" upper="2.443" />
+        <limit effort="0.95" velocity="8.48" acceleration="20.0" lower="-2.47" upper="2.443" />
         <joint_properties friction="0.0" />
     </joint>
@@ -169,5 +169,5 @@
         <child link="thumb_middle_phalanx" />
         <axis xyz="0 0 -1" />
-        <limit effort="0.95" velocity="8.48" lower="-1.20" upper="1.90" />
+        <limit effort="0.95" velocity="8.48" acceleration="20.0" lower="-1.20" upper="1.90" />
         <joint_properties friction="0.0" />
     </joint>
@@ -178,5 +178,5 @@
         <child link="thumb_distal_phalanx" />
         <axis xyz="0 0 -1" />
-        <limit effort="0.95" velocity="8.48" lower="-1.34" upper="1.88" />
+        <limit effort="0.95" velocity="8.48" acceleration="20.0" lower="-1.34" upper="1.88" />
         <joint_properties friction="0.0" />
     </joint>

File: leap_moveit/config/leap.ros2_control.xacro (robot description, xacro)
@@ -1,5 +1,5 @@
 <?xml version="1.0"?>
 <robot xmlns:xacro="http://www.ros.org/wiki/xacro">
-    <xacro:macro name="onshape_ros2_control" params="name initial_positions_file">
+    <xacro:macro name="leap_ros2_control" params="name initial_positions_file">
         <xacro:property name="initial_positions" value="${xacro.load_yaml(initial_positions_file)['initial_positions']}"/>
         <ros2_control name="${name}" type="system">
@@ -8,163 +8,131 @@
                 <plugin>mock_components/GenericSystem</plugin>
             </hardware>
-            <joint name="0">
+            <joint name="index_pip_flex_joint">
                 <command_interface name="position"/>
-                <command_interface name="velocity"/>
                 <command_interface name="effort"/>
                 <state_interface name="position">
-                  <param name="initial_value">${initial_positions['0']}</param>
+                  <param name="initial_value">${initial_positions['index_pip_flex_joint']}</param>
                 </state_interface>
                 <state_interface name="velocity"/>
-                <state_interface name="effort"/>
             </joint>
-            <joint name="1">
+            <joint name="index_pip_abb_joint">
                 <command_interface name="position"/>
-                <command_interface name="velocity"/>
                 <command_interface name="effort"/>
                 <state_interface name="position">
-                  <param name="initial_value">${initial_positions['1']}</param>
+                  <param name="initial_value">${initial_positions['index_pip_abb_joint']}</param>
                 </state_interface>
                 <state_interface name="velocity"/>
-                <state_interface name="effort"/>
             </joint>
-            <joint name="2">
+            <joint name="index_mcp_joint">
                 <command_interface name="position"/>
-                <command_interface name="velocity"/>
                 <command_interface name="effort"/>
                 <state_interface name="position">
-                  <param name="initial_value">${initial_positions['2']}</param>
+                  <param name="initial_value">${initial_positions['index_mcp_joint']}</param>
                 </state_interface>
                 <state_interface name="velocity"/>
-                <state_interface name="effort"/>
             </joint>
-            <joint name="3">
+            <joint name="index_dip_joint">
                 <command_interface name="position"/>
-                <command_interface name="velocity"/>
                 <command_interface name="effort"/>
                 <state_interface name="position">
-                  <param name="initial_value">${initial_positions['3']}</param>
+                  <param name="initial_value">${initial_positions['index_dip_joint']}</param>
                 </state_interface>
                 <state_interface name="velocity"/>
-                <state_interface name="effort"/>
             </joint>
-            <joint name="12">
+            <joint name="middle_pip_flex_joint">
                 <command_interface name="position"/>
-                <command_interface name="velocity"/>
                 <command_interface name="effort"/>
                 <state_interface name="position">
-                  <param name="initial_value">${initial_positions['12']}</param>
+                  <param name="initial_value">${initial_positions['middle_pip_flex_joint']}</param>
                 </state_interface>
                 <state_interface name="velocity"/>
-                <state_interface name="effort"/>
             </joint>
-            <joint name="13">
+            <joint name="middle_pip_abb_joint">
                 <command_interface name="position"/>
-                <command_interface name="velocity"/>
                 <command_interface name="effort"/>
                 <state_interface name="position">
-                  <param name="initial_value">${initial_positions['13']}</param>
+                  <param name="initial_value">${initial_positions['middle_pip_abb_joint']}</param>
                 </state_interface>
                 <state_interface name="velocity"/>
-                <state_interface name="effort"/>
             </joint>
-            <joint name="14">
+            <joint name="middle_mcp_joint">
                 <command_interface name="position"/>
-                <command_interface name="velocity"/>
                 <command_interface name="effort"/>
                 <state_interface name="position">
-                  <param name="initial_value">${initial_positions['14']}</param>
+                  <param name="initial_value">${initial_positions['middle_mcp_joint']}</param>
                 </state_interface>
                 <state_interface name="velocity"/>
-                <state_interface name="effort"/>
             </joint>
-            <joint name="15">
+            <joint name="middle_dip_joint">
                 <command_interface name="position"/>
-                <command_interface name="velocity"/>
                 <command_interface name="effort"/>
                 <state_interface name="position">
-                  <param name="initial_value">${initial_positions['15']}</param>
+                  <param name="initial_value">${initial_positions['middle_dip_joint']}</param>
                 </state_interface>
                 <state_interface name="velocity"/>
-                <state_interface name="effort"/>
             </joint>
-            <joint name="4">
+            <joint name="ring_pip_flex_joint">
                 <command_interface name="position"/>
-                <command_interface name="velocity"/>
                 <command_interface name="effort"/>
                 <state_interface name="position">
-                  <param name="initial_value">${initial_positions['4']}</param>
+                  <param name="initial_value">${initial_positions['ring_pip_flex_joint']}</param>
                 </state_interface>
                 <state_interface name="velocity"/>
-                <state_interface name="effort"/>
             </joint>
-            <joint name="5">
+            <joint name="ring_pip_abb_joint">
                 <command_interface name="position"/>
-                <command_interface name="velocity"/>
                 <command_interface name="effort"/>
                 <state_interface name="position">
-                  <param name="initial_value">${initial_positions['5']}</param>
+                  <param name="initial_value">${initial_positions['ring_pip_abb_joint']}</param>
                 </state_interface>
                 <state_interface name="velocity"/>
-                <state_interface name="effort"/>
             </joint>
-            <joint name="6">
+            <joint name="ring_mcp_joint">
                 <command_interface name="position"/>
-                <command_interface name="velocity"/>
                 <command_interface name="effort"/>
                 <state_interface name="position">
-                  <param name="initial_value">${initial_positions['6']}</param>
+                  <param name="initial_value">${initial_positions['ring_mcp_joint']}</param>
                 </state_interface>
                 <state_interface name="velocity"/>
-                <state_interface name="effort"/>
             </joint>
-            <joint name="7">
+            <joint name="ring_dip_joint">
                 <command_interface name="position"/>
-                <command_interface name="velocity"/>
                 <command_interface name="effort"/>
                 <state_interface name="position">
-                  <param name="initial_value">${initial_positions['7']}</param>
+                  <param name="initial_value">${initial_positions['ring_dip_joint']}</param>
                 </state_interface>
                 <state_interface name="velocity"/>
-                <state_interface name="effort"/>
             </joint>
-            <joint name="8">
+            <joint name="thumb_cmc_abb_joint">
                 <command_interface name="position"/>
-                <command_interface name="velocity"/>
                 <command_interface name="effort"/>
                 <state_interface name="position">
-                  <param name="initial_value">${initial_positions['8']}</param>
+                  <param name="initial_value">${initial_positions['thumb_cmc_abb_joint']}</param>
                 </state_interface>
                 <state_interface name="velocity"/>
-                <state_interface name="effort"/>
             </joint>
-            <joint name="9">
+            <joint name="thumb_cmc_flex_joint">
                 <command_interface name="position"/>
-                <command_interface name="velocity"/>
                 <command_interface name="effort"/>
                 <state_interface name="position">
-                  <param name="initial_value">${initial_positions['9']}</param>
+                  <param name="initial_value">${initial_positions['thumb_cmc_flex_joint']}</param>
                 </state_interface>
                 <state_interface name="velocity"/>
-                <state_interface name="effort"/>
             </joint>
-            <joint name="10">
+            <joint name="thumb_mcp_joint">
                 <command_interface name="position"/>
-                <command_interface name="velocity"/>
                 <command_interface name="effort"/>
                 <state_interface name="position">
-                  <param name="initial_value">${initial_positions['10']}</param>
+                  <param name="initial_value">${initial_positions['thumb_mcp_joint']}</param>
                 </state_interface>
                 <state_interface name="velocity"/>
-                <state_interface name="effort"/>
             </joint>
-            <joint name="11">
+            <joint name="thumb_ip_joint">
                 <command_interface name="position"/>
-                <command_interface name="velocity"/>
                 <command_interface name="effort"/>
                 <state_interface name="position">
-                  <param name="initial_value">${initial_positions['11']}</param>
+                  <param name="initial_value">${initial_positions['thumb_ip_joint']}</param>
                 </state_interface>
                 <state_interface name="velocity"/>
-                <state_interface name="effort"/>
             </joint>
         </ros2_control>

Commit message: Created mesh collision that are convex hull approximations of major parts  of the links. This transformation was done in blender, and the blender files are also stored

File: leap_description/assets/leap_hand/finger.xacro (robot description, xacro)
@@ -12,5 +12,5 @@
                 <material name="proximal_phalanx_1_material">
                     <color
-                        rgba="0 0 0 1.0" />
+                        rgba="0.0 0 0 1.0" />
                 </material>
             </visual>
@@ -20,5 +20,13 @@
                     rpy="0 0 0" />
                 <geometry>
-                    <mesh filename="package://leap_description/assets/leap_hand/proximal_phalanx_1.stl" />
+                    <mesh filename="package://leap_description/assets/leap_hand/proximal_phalanx_1_collision.stl" />
+                </geometry>
+            </collision>
+            <collision>
+                <origin
+                    xyz="-0.0 0.007 0.014"
+                    rpy="0 0 0" />
+                <geometry>
+                    <box size="0.0225 0.03 0.035"/>
                 </geometry>
             </collision>
@@ -40,5 +48,5 @@
                 <material name="proximal_phalanx_2_material">
                     <color
-                        rgba="0 0 0 1.0" />
+                        rgba="0.0 0 0 1.0" />
                 </material>
             </visual>
@@ -48,5 +56,5 @@
                     rpy="-1.570796326794896558 -1.570796326794896336 0" />
                 <geometry>
-                    <mesh filename="package://leap_description/assets/leap_hand/proximal_phalanx_2.stl" />
+                    <mesh filename="package://leap_description/assets/leap_hand/proximal_phalanx_2_collision.stl" />
                 </geometry>
             </collision>
@@ -68,5 +76,5 @@
                 <material name="middle_phalanx_material">
                     <color
-                        rgba="0 0 0 1.0" />
+                        rgba="0.0 0 0 1.0" />
                 </material>
             </visual>
@@ -76,5 +84,5 @@
                     rpy="-3.141592653589793116 0 0" />
                 <geometry>
-                    <mesh filename="package://leap_description/assets/leap_hand/middle_phalanx.stl" />
+                    <mesh filename="package://leap_description/assets/leap_hand/middle_phalanx_collision.stl" />
                 </geometry>
             </collision>
@@ -104,5 +112,5 @@
                     rpy="3.141592653589793116 0 0" />
                 <geometry>
-                    <mesh filename="package://leap_description/assets/leap_hand/distal_phalanx.stl" />
+                    <mesh filename="package://leap_description/assets/leap_hand/distal_phalanx_collision.stl" />
                 </geometry>
             </collision>

File: leap_description/assets/leap_hand/robot.urdf.xacro (robot description, xacro)
@@ -18,5 +18,5 @@
                 rpy="0 -0 0" />
             <geometry>
-                <mesh filename="package://leap_description/assets/leap_hand/palm_lower.stl" />
+                <mesh filename="package://leap_description/assets/leap_hand/palm_lower_collision.stl" />
             </geometry>
         </collision>
@@ -52,5 +52,5 @@
                 rpy="-1.570796326794896558 -1.570796326794896336 0" />
             <geometry>
-                <mesh filename="package://leap_description/assets/leap_hand/proximal_phalanx_2.stl" />
+                <mesh filename="package://leap_description/assets/leap_hand/proximal_phalanx_2_collision.stl" />
             </geometry>
         </collision>
@@ -80,5 +80,5 @@
                 rpy="1.570796326794896558 0 0" />
             <geometry>
-                <mesh filename="package://leap_description/assets/leap_hand/thumb_semi_palm.stl" />
+                <mesh filename="package://leap_description/assets/leap_hand/thumb_semi_palm_collision.stl" />
             </geometry>
         </collision>
@@ -107,5 +107,5 @@
             <geometry>
                 <mesh
-                    filename="package://leap_description/assets/leap_hand/thumb_middle_phalanx.stl" />
+                    filename="package://leap_description/assets/leap_hand/thumb_middle_phalanx_collision.stl" />
             </geometry>
         </collision>
@@ -135,5 +135,5 @@
             <geometry>
                 <mesh
-                    filename="package://leap_description/assets/leap_hand/thumb_distal_phalanx.stl" />
+                    filename="package://leap_description/assets/leap_hand/thumb_distal_phalanx_collision.stl" />
             </geometry>
         </collision>
