Commit message: Corrected the URDF of the robot (one thumb joint was incorrectly rotated 180 degrees)

File: leap_description/assets/leap_hand/finger.xacro (robot description, xacro)
@@ -128,5 +128,5 @@
             <child link="${finger}_proximal_phalanx_1" />
             <axis xyz="0 0 -1" />
-            <limit effort="0.95" velocity="8.48" acceleration="20.0" lower="-0.314" upper="2.23" />
+            <limit effort="0.95" velocity="8.48" acceleration="20.0" lower="-0.31416" upper="2.3038" />
             <joint_properties friction="0.0" />
         </joint>
@@ -137,5 +137,5 @@
             <child link="${finger}_proximal_phalanx_2" />
             <axis xyz="0 0 -1" />
-            <limit effort="0.95" velocity="8.48" acceleration="20.0" lower="-1.047" upper="1.047" />
+            <limit effort="0.95" velocity="8.48" acceleration="20.0" lower="-1.378810" upper="1.378810"/>
             <joint_properties friction="0.0" />
         </joint>
@@ -146,5 +146,5 @@
             <child link="${finger}_middle_phalanx" />
             <axis xyz="0 0 -1" />
-            <limit effort="0.95" velocity="8.48" acceleration="20.0" lower="-0.506" upper="1.885" />
+            <limit effort="0.95" velocity="8.48" acceleration="20.0" lower="-0.45379" upper="2.44346" />
             <joint_properties friction="0.0" />
         </joint>
@@ -156,5 +156,5 @@
             <child link="${finger}_distal_phalanx" />
             <axis xyz="0 0 -1" />
-            <limit effort="0.95" velocity="8.48" acceleration="20.0" lower="-0.366" upper="2.042" />
+            <limit effort="0.95" velocity="8.48" acceleration="20.0" lower="-0.3491" upper="1.867502" />
             <joint_properties friction="0.0" />
         </joint>

File: leap_description/assets/leap_hand/robot.urdf.xacro (robot description, xacro)
@@ -151,14 +151,14 @@
         <child link="thumb_semi_palm_1" />
         <axis xyz="0 0 -1" />
-        <limit effort="0.95" velocity="8.48" acceleration="20.0" lower="-0.349" upper="2.094" />
+        <limit effort="0.95" velocity="8.48" acceleration="20.0" lower="-0.38397" upper="2.02458" />
         <joint_properties friction="0.0" />
     </joint>
     <joint name="thumb_cmc_flex_joint" type="revolute">
         <origin xyz="0 0.0143 -0.013"
-            rpy="1.5707963267948958919 1.5707963267948958919 0" />
+            rpy="1.5707963267948958919 -1.5707963267948958919 0" />
         <parent link="thumb_semi_palm_1" />
         <child link="thumb_semi_palm_2" />
         <axis xyz="0 0 -1" />
-        <limit effort="0.95" velocity="8.48" acceleration="20.0" lower="-2.47" upper="2.443" />
+        <limit effort="0.95" velocity="8.48" acceleration="20.0" lower="-0.7854" upper="1.570796" />
         <joint_properties friction="0.0" />
     </joint>
@@ -169,5 +169,5 @@
         <child link="thumb_middle_phalanx" />
         <axis xyz="0 0 -1" />
-        <limit effort="0.95" velocity="8.48" acceleration="20.0" lower="-1.20" upper="1.90" />
+        <limit effort="0.95" velocity="8.48" acceleration="20.0" lower="-0.34906" upper="1.7453" />
         <joint_properties friction="0.0" />
     </joint>
@@ -178,5 +178,5 @@
         <child link="thumb_distal_phalanx" />
         <axis xyz="0 0 -1" />
-        <limit effort="0.95" velocity="8.48" acceleration="20.0" lower="-1.34" upper="1.88" />
+        <limit effort="0.95" velocity="8.48" acceleration="20.0" lower="-0.7854" upper="1.93731" />
         <joint_properties friction="0.0" />
     </joint>

File: leap_moveit/config/leap.ros2_control.xacro (robot description, xacro)
@@ -5,5 +5,6 @@
         <ros2_control name="${name}" type="system">
             <hardware>
-              <plugin>mock_components/GenericSystem</plugin>
+                <!-- By default, set up controllers for simulation. This won't work on real hardware -->
+                <plugin>mock_components/GenericSystem</plugin>
             </hardware>
             <joint name="index_pip_flex_joint">

File: leap_moveit/config/leap.urdf.xacro (robot description, xacro)
@@ -2,21 +2,8 @@
 <robot xmlns:xacro="http://www.ros.org/wiki/xacro" name="leap">
     <xacro:arg name="initial_positions_file" default="initial_positions.yaml" />
-    <xacro:arg name="use_gazebo" default="false" />
     <!-- Import leap urdf file -->
     <xacro:include filename="$(find leap_description)/assets/leap_hand/robot.urdf.xacro" />
     <!-- Import control_xacro -->
-    <xacro:if value="$(arg use_gazebo)">
-        <xacro:include filename="leap.gz_control.xacro" />
-        <xacro:leap_gz_control name="GazeboSimSystem" initial_positions_file="$(arg initial_positions_file)"/>
-        <gazebo>
-            <plugin filename="libgz_ros2_control-system.so" name="gz_ros2_control::GazeboSimROS2ControlPlugin">
-                <!-- <parameters>$(arg controllers_yaml)</parameters> -->
-                <parameters>/home/joel/distrobox/ros2-ubuntu/leap_ws/src/leap_control/leap_sim/config/leap_controller.yaml</parameters>
-            </plugin>
-        </gazebo>
-    </xacro:if>
-    <xacro:unless value="$(arg use_gazebo)">
-        <xacro:include filename="leap.ros2_control.xacro" />
-        <xacro:leap_ros2_control name="FakeSystem" initial_positions_file="$(arg initial_positions_file)"/>
-    </xacro:unless>
+    <xacro:include filename="leap.ros2_control.xacro" />
+    <xacro:leap_ros2_control name="FakeSystem" initial_positions_file="$(arg initial_positions_file)"/>
 </robot>

Commit message: Solved the problem with the collision between consecutive links in webots by changing the meshes

File: leap_description/assets/leap_hand/finger.xacro (robot description, xacro)
@@ -8,5 +8,5 @@
                     rpy="0 0 0" />
                 <geometry>
-                    <mesh filename="package://leap_description/assets/leap_hand/proximal_phalanx_1.stl" />
+                    <mesh filename="package://leap_description/assets/leap_hand/proximal_phalanx_1_2k.stl" />
                 </geometry>
                 <material name="proximal_phalanx_1_material">
@@ -20,5 +20,5 @@
                     rpy="0 0 0" />
                 <geometry>
-                    <mesh filename="package://leap_description/assets/leap_hand/proximal_phalanx_1_collision.stl" />
+                    <mesh filename="package://leap_description/assets/leap_hand/proximal_phalanx_1_2k_collision.stl" />
                 </geometry>
             </collision>
@@ -44,5 +44,5 @@
                     rpy="-1.570796326794896558 -1.570796326794896336 0" />
                 <geometry>
-                    <mesh filename="package://leap_description/assets/leap_hand/proximal_phalanx_2.stl" />
+                    <mesh filename="package://leap_description/assets/leap_hand/proximal_phalanx_2_2k.stl" />
                 </geometry>
                 <material name="proximal_phalanx_2_material">
@@ -56,5 +56,5 @@
                     rpy="-1.570796326794896558 -1.570796326794896336 0" />
                 <geometry>
-                    <mesh filename="package://leap_description/assets/leap_hand/proximal_phalanx_2_collision.stl" />
+                    <mesh filename="package://leap_description/assets/leap_hand/proximal_phalanx_2_2k_collision.stl" />
                 </geometry>
             </collision>
@@ -72,5 +72,5 @@
                     rpy="-3.141592653589793116 0 0" />
                 <geometry>
-                    <mesh filename="package://leap_description/assets/leap_hand/middle_phalanx.stl" />
+                    <mesh filename="package://leap_description/assets/leap_hand/middle_phalanx_2k.stl" />
                 </geometry>
                 <material name="middle_phalanx_material">
@@ -84,5 +84,5 @@
                     rpy="-3.141592653589793116 0 0" />
                 <geometry>
-                    <mesh filename="package://leap_description/assets/leap_hand/middle_phalanx_collision.stl" />
+                    <mesh filename="package://leap_description/assets/leap_hand/middle_phalanx_2k_collision.stl" />
                 </geometry>
             </collision>
@@ -100,5 +100,5 @@
                     rpy="3.141592653589793116 0 0" />
                 <geometry>
-                    <mesh filename="package://leap_description/assets/leap_hand/distal_phalanx.stl" />
+                    <mesh filename="package://leap_description/assets/leap_hand/distal_phalanx_1k.stl" />
                 </geometry>
                 <material name="distal_phalanx_material">
@@ -112,5 +112,5 @@
                     rpy="3.141592653589793116 0 0" />
                 <geometry>
-                    <mesh filename="package://leap_description/assets/leap_hand/distal_phalanx_collision.stl" />
+                    <mesh filename="package://leap_description/assets/leap_hand/distal_phalanx_1k_collision.stl" />
                 </geometry>
             </collision>

File: leap_description/assets/leap_hand/robot.urdf.xacro (robot description, xacro)
@@ -7,5 +7,5 @@
                 rpy="0 -0 0" />
             <geometry>
-                <mesh filename="package://leap_description/assets/leap_hand/palm_lower.stl" />
+                <mesh filename="package://leap_description/assets/leap_hand/palm_lower_3k.stl" />
             </geometry>
             <material name="palm_lower_material">
@@ -18,5 +18,5 @@
                 rpy="0 -0 0" />
             <geometry>
-                <mesh filename="package://leap_description/assets/leap_hand/palm_lower_collision.stl" />
+                <mesh filename="package://leap_description/assets/leap_hand/palm_lower_3k_collision.stl" />
             </geometry>
         </collision>
@@ -40,5 +40,5 @@
                 rpy="-1.570796326794896558 -1.570796326794896336 0" />
             <geometry>
-                <mesh filename="package://leap_description/assets/leap_hand/proximal_phalanx_2.stl" />
+                <mesh filename="package://leap_description/assets/leap_hand/proximal_phalanx_2_2k.stl" />
             </geometry>
             <material name="thumb_semi_palm_2_material">
@@ -52,5 +52,5 @@
                 rpy="-1.570796326794896558 -1.570796326794896336 0" />
             <geometry>
-                <mesh filename="package://leap_description/assets/leap_hand/proximal_phalanx_2_collision.stl" />
+                <mesh filename="package://leap_description/assets/leap_hand/proximal_phalanx_2_2k_collision.stl" />
             </geometry>
         </collision>
@@ -68,5 +68,5 @@
                 rpy="1.570796326794896558 0 0" />
             <geometry>
-                <mesh filename="package://leap_description/assets/leap_hand/thumb_semi_palm.stl" />
+                <mesh filename="package://leap_description/assets/leap_hand/thumb_semi_palm_1k.stl" />
             </geometry>
             <material name="thumb_semi_palm_2_material">
@@ -80,5 +80,5 @@
                 rpy="1.570796326794896558 0 0" />
             <geometry>
-                <mesh filename="package://leap_description/assets/leap_hand/thumb_semi_palm_collision.stl" />
+                <mesh filename="package://leap_description/assets/leap_hand/thumb_semi_palm_1k_collision.stl" />
             </geometry>
         </collision>
@@ -95,5 +95,5 @@
             <geometry>
                 <mesh
-                    filename="package://leap_description/assets/leap_hand/thumb_middle_phalanx.stl" />
+                    filename="package://leap_description/assets/leap_hand/thumb_middle_phalanx_3k.stl" />
             </geometry>
             <material name="thumb_middle_phalanx_material">
@@ -107,5 +107,5 @@
             <geometry>
                 <mesh
-                    filename="package://leap_description/assets/leap_hand/thumb_middle_phalanx_collision.stl" />
+                    filename="package://leap_description/assets/leap_hand/thumb_middle_phalanx_3k_collision.stl" />
             </geometry>
         </collision>
@@ -123,5 +123,5 @@
             <geometry>
                 <mesh
-                    filename="package://leap_description/assets/leap_hand/thumb_distal_phalanx.stl" />
+                    filename="package://leap_description/assets/leap_hand/thumb_distal_phalanx_1k.stl" />
             </geometry>
             <material name="thumb_distal_phalanx_material">
@@ -135,5 +135,5 @@
             <geometry>
                 <mesh
-                    filename="package://leap_description/assets/leap_hand/thumb_distal_phalanx_collision.stl" />
+                    filename="package://leap_description/assets/leap_hand/thumb_distal_phalanx_1k_collision.stl" />
             </geometry>
         </collision>
