Commit message: Solved instalbility in Webots simulation

File: leap_description/urdf/robot.urdf (robot description, URDF)
Before this commit: robot leap, 17 links, 16 joints
Links:
- link index_distal_phalanx: geometry collision mesh filename=package://leap_description/assets/leap_hand/distal_phalanx_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; visual mesh filename=package://leap_description/assets/leap_hand/distal_phalanx.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
- link index_middle_phalanx: geometry collision mesh filename=package://leap_description/assets/leap_hand/middle_phalanx_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; visual mesh filename=package://leap_description/assets/leap_hand/middle_phalanx.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
- link index_proximal_phalanx_1: geometry collision box size=0.0225 0.03 0.035; collision mesh filename=package://leap_description/assets/leap_hand/proximal_phalan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
- link middle_distal_phalanx: geometry collision mesh filename=package://leap_description/assets/leap_hand/distal_phalanx_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; visual mesh filename=package://leap_description/assets/leap_hand/distal_phalanx.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
- link middle_middle_phalanx: geometry collision mesh filename=package://leap_description/assets/leap_hand/middle_phalanx_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; visual mesh filename=package://leap_description/assets/leap_hand/middle_phalanx.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
- link middle_proximal_phalanx_1: geometry collision box size=0.0225 0.03 0.035; collision mesh filename=package://leap_description/assets/leap_hand/proximal_phalan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
- link palm_lower: geometry collision mesh filename=package://leap_description/assets/leap_hand/palm_lower_coll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; visual mesh filename=package://leap_description/assets/leap_hand/palm_lower.stl
- link ring_distal_phalanx: geometry collision mesh filename=package://leap_description/assets/leap_hand/distal_phalanx_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; visual mesh filename=package://leap_description/assets/leap_hand/distal_phalanx.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
- link ring_middle_phalanx: geometry collision mesh filename=package://leap_description/assets/leap_hand/middle_phalanx_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; visual mesh filename=package://leap_description/assets/leap_hand/middle_phalanx.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
- link ring_proximal_phalanx_1: geometry collision box size=0.0225 0.03 0.035; collision mesh filename=package://leap_description/assets/leap_hand/proximal_phalan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
